File: hardware/hackaday-sao-m5stack-atoms3.kicad_pcb (KiCad board)
At the start: 2 copper layers, 46 x 45 mm, 4 parts, among them J2 Conn_02x03_Odd_Even

Commit message: Added version 0.1
Other:
- board text added: "M5Stack Atom-SAO"
- board text removed: "M5Stach Atom-SAO"

Commit message: Project updated
Routing:
- net GPIO2: track 36.5 -> 32.4 mm
- net GPIO1: track 38.9 -> 35.8 mm
- net SCL: track 34.1 -> 32.3 mm
- net GND: vias 20 -> 30
Other:
- board text added: "SAO"
